File: ReadaptTTGO/_autosave-ReadaptTTGO.kicad_pcb (KiCad board)
At the start: 2 copper layers, 80 x 115 mm, 101 parts, among them J1 USB_B_Micro, J2 Conn_01x02_Shielded, J3 Micro_SD_Card, J4 Conn_01x13_Female, J5 Conn_01x13_Female, SW1 SW_SPDT, SW2 SW_Push, U1 CP2102N-A01-GQFN24, U2 ESP32, U3 EMH3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

Commit message: Comienzo PCB
Parts:
- moved D3 203.6 mm to (225.5, 135.5), turned to 90 degrees
- moved C3 191.5 mm to (245.9, 60.5)
- moved C7 191.5 mm to (248.2, 60.4)
- moved R10 191.5 mm to (250.5, 60.4)
- moved D4 186.4 mm to (225.5, 130.0), turned to 90 degrees
- moved SW1 180.7 mm to (231.5, 122.5), turned to 90 degrees
- moved J1 173.6 mm to (233.5, 134.5), turned to 90 degrees
- moved C28 172.8 mm to (219.0, 141.0)
- moved R29 172.7 mm to (216.5, 141.0), turned to 180 degrees
- moved SW2 171.3 mm to (220.5, 147.0), turned to 180 degrees
- moved U4 166.0 mm to (204.5, 137.0), turned to 270 degrees
- moved U3 164.5 mm to (191.5, 103.5), turned to 180 degrees
- moved D2 149.7 mm to (212.0, 116.5)
- moved FL1 149.0 mm to (204.5, 115.0), turned to 180 degrees
- moved U6 136.9 mm to (202.5, 129.5)
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