File: ReadaptTTGO/microesp32.sch (KiCad schematic (older format))
At the start: 1 part, among them U2 ESP32

Commit message: Primer aproximacion.
Parts:
- added AE?: Antenna_Chip, symbol Device:Antenna_Chip
- added C? (x5): C, symbol Device:C
- added C?: 5.6pF, symbol Device:C
- added C? (x2): 270pF, symbol Device:C
- added C?: 1uF, symbol Device:C
- added D?: LED RED, symbol Device:LED
- added D?: LED GREEN, symbol Device:LED
- added D? (x6): ULC0511C, symbol Device:D_TVS
- added H? (x3): MountingHole, symbol Mechanical:MountingHole
- added J? (x2): Conn_01x13_Female, symbol Connector:Conn_01x13_Female
- added J?: Micro_SD_Card, symbol Connector:Micro_SD_Card
- added R?: 10K, symbol Device:R
- added R?: 0R, symbol Device:R
- added R? (x2): 470, symbol Device:R
- added R? (x4): 22, symbol Device:R
- added R? (x2): 2K, symbol Device:R
- added R? (x5): NC, symbol Device:R
- added SW?: SW_Push, symbol Switch:SW_Push
Connections:
- net +3V3: now reaches U2.1 (VDDA)
- net +3V3: now also U2.19 (VDD3P3_RTC), U2.3 (VDD3P3), U2.37 (VDD3P3_CPU), U2.4 (VDD3P3), U2.43 (VDDA), U2.46 (VDDA), C?.1, C?.1, C?.1, J?.4 (VDD), R?.1, R?.1, R?.2, R?.2, R?.2, R?.2, R?.2
- net IO34: now reaches U2.10 (VDET_1)
- net IO34: now also J?.10 (Pin_10)
- net IO35: now reaches U2.11 (VDET_2)
- net IO35: now also J?.9 (Pin_9)
- net IO32: now reaches U2.12 (32K_XP)
- net IO32: now also R?.1
- net IO33: now reaches U2.13 (32K_XN)
- net IO33: now also R?.1
- net IO25: now reaches U2.14 (GPIO25)
- net IO25: now also J?.1 (Pin_1), R?.2
- net IO26: now reaches U2.15 (GPIO26)
- net IO27: now reaches U2.16 (GPIO27)
- net CLK-SCK-IO14: now reaches U2.17 (MTMS)
- net CLK-SCK-IO14: now also D?.1 (A1), J?.5 (CLK), J?.8 (Pin_8), R?.1
- net SD2-IO12: now reaches U2.18 (MTDI)
- net SD2-IO12: now also D?.1 (A1), J?.1 (DAT2), J?.7 (Pin_7), R?.2
- net at U2.2 (LNA_IN): now also C?.1, C?.1
- net SD3-CS-IO13: now reaches U2.20 (MTCK)
- net SD3-CS-IO13: now also D?.2 (A2), J?.2 (DAT3/CD), J?.6 (Pin_6), R?.1
- net CMD-MOSI-IO15: now reaches U2.21 (MTDO)
- net CMD-MOSI-IO15: now also D?.2 (A2), J?.3 (CMD), J?.5 (Pin_5)
- net SD0-MISO-IO2: now reaches U2.22 (GPIO2)
- net SD0-MISO-IO2: now also D?.1 (A1), J?.4 (Pin_4), J?.7 (DAT0), R?.1
- net IO0: now reaches U2.23 (GPIO0)
- net IO0: now also J?.3 (Pin_3)
- net SD1-IO4: now reaches U2.24 (GPIO4)
- net SD1-IO4: now also D?.2 (A2), J?.2 (Pin_2), J?.8 (DAT1), R?.1
- net IO5: now reaches U2.34 (GPIO5)
- net IO18: now reaches U2.35 (GPIO18)
- net IO23: now reaches U2.36 (GPIO23)
- net IO23: now also J?.9 (Pin_9)
- net IO19: now reaches U2.38 (GPIO19)
- net IO22: now reaches U2.39 (GPIO22)
- net IO22: now also J?.10 (Pin_10), R?.1
- net RDX: now reaches U2.40 (U0RXD)
- net TXD: now reaches U2.41 (U0TXD)
- net TXD: now also J?.12 (Pin_12), R?.1
- net IO21: now reaches U2.42 (GPIO21)
- net IO21: now also J?.13 (Pin_13), R?.1
- net GND: now reaches U2.49 (GND_PAD)
- net GND: now also AE?.1 (FEED), C?.2, C?.2, C?.2, C?.2, C?.2, C?.2, D?.1 (A1), D?.1 (A1), D?.1 (A1), D?.1 (K), D?.1 (K), D?.2 (A2), D?.2 (A2), D?.2 (A2), J?.2 (Pin_2), J?.4 (Pin_4), J?.6 (VSS), J?.9 (SHIELD), SW?.1
- net S_VP: now reaches U2.5 (SENSOR_VP)
- net S_VP: now also C?.1, J?.13 (Pin_13)
- net SENSOR_CAPP: now reaches U2.6 (SENSOR_CAPP)
- net SENSOR_CAPP: now also C?.2
- net SENSOR_CAPN: now reaches U2.7 (SENSOR_CAPN)
- net SENSOR_CAPN: now also C?.2
- net S_VN: now reaches U2.8 (SENSOR_VN)
- net S_VN: now also C?.1, J?.12 (Pin_12)
- net RST_EN: now reaches U2.9 (CHIP_PU)
- net RST_EN: now also J?.11 (Pin_11)
- new net: AE?.2 (PCB_Trace), C?.1, C?.2
- new net: R?.2, SW?.2
- new net: D?.2 (A), R?.1 (x2)
- new net +3.3VP: J?.3 (Pin_3)
- new net +5V: J?.1 (Pin_1)
- new net D0: R?.2
- new net D1: R?.2
- new net HPDIO1: J?.6 (Pin_6), R?.2
- new net HPDIO2: J?.7 (Pin_7), R?.2
- new net RS_EN: C?.1, R?.1, R?.2
- new net RXD: J?.11 (Pin_11), R?.1
- new net U0RXD: R?.2, R?.2
- new net asdsa: J?.8 (Pin_8)
- no-connect marks 0 -> 1
Other:
- moved on the sheet: U2

Commit message: Anotacciones
Parts:
- gave numbers to parts that had none: 40

Commit message: ERC completo
Connections:
- net RDX is gone; now on net RXD: U2.40 (U0RXD)
- net asdsa is gone; now on net IO19: J4.8 (Pin_8)
- no-connect marks 1 -> 14
Changed lines of the file:
@@
 Wire Wire Line
 	5700 3000 5700 3100
-Wire Wire Line
-	2550 2900 5700 2900
 $Comp
 L Device:C C21
@@
 TXD
 Text Label 7600 1300 1    50   ~ 0
-RDX
+RXD
 $Comp
 L power:+3V3 #PWR0167
@@
 Wire Wire Line
 	8800 3000 9450 3000
-Text Label 9450 3000 0    50   ~ 0
-IO5
 Text Label 9450 2800 0    50   ~ 0
 IO23
@@
 	1350 7000 1000 7000
 Text Label 1000 7000 0    50   ~ 0
-asdsa
+IO19
 Text HLabel 1000 6900 0    50   Input ~ 0
 HPDIO2
@@
 Wire Wire Line
 	2600 5450 3100 5450
+NoConn ~ 1000 6700
+NoConn ~ 8800 3900
+NoConn ~ 8800 3700
+NoConn ~ 8800 3600
+NoConn ~ 8800 3500
+NoConn ~ 8800 3400
+NoConn ~ 8800 3300
+NoConn ~ 8800 3200
+NoConn ~ 8800 3100
+NoConn ~ 6800 1900
+NoConn ~ 6900 1900
+NoConn ~ 7100 1900
+NoConn ~ 7200 1900
+Text Label 9450 3000 0    50   ~ 0
+IO5
+Wire Wire Line
+	2550 2900 5700 2900
 $EndSCHEMATC

Commit message: Añadidos Footprints
Parts:
- C20, C21, C22, C23, C24, C25, C27, C28: footprint (none) -> Capacitor_SMD:C_01005_0402Metric
- C26: footprint (none) -> Capacitor_SMD:C_0201_0603Metric
- D10, D11, D12, D7, D8, D9: footprint (none) -> Diode_SMD:D_01005_0402Metric
- D13, D14: footprint (none) -> LED_SMD:LED_0201_0603Metric
- H1, H2, H3: footprint (none) -> Fiducial:Fiducial_1mm_Mask2mm
- J3: footprint (none) -> Connector_Card:microSD_HC_Hirose_DM3D-SF
- J4, J5: footprint (none) -> TerminalBlock_Phoenix:TerminalBlock_Phoenix_PT-1,5-13-5.0-H_1x13_P5.00mm_Horizontal
- R22, R23, R24, R25, R26, R27, R28, R29, R30, R31, R32, R33, R34, R35, R36: footprint (none) -> Resistor_SMD:R_01005_0402Metric
- SW2: footprint (none) -> Button_Switch_SMD:SW_Push_1P1T_NO_6x6mm_H9.5mm
- U2: footprint (none) -> Package_DFN_QFN:UQFN-48-1EP_6x6mm_P0.4mm_EP4.45x4.45mm
Changed lines of the file:
@@
 F 0 "U2" H 8844 2303 60  0000 L CNN
 F 1 "ESP32" H 8844 2197 60  0000 L CNN
-F 2 "" H 5700 2800 50  0001 C CNN
+F 2 "Package_DFN_QFN:UQFN-48-1EP_6x6mm_P0.4mm_EP4.45x4.45mm" H 5700 2800 50  0001 C CNN
 F 3 "https://espressif.com/sites/default/files/documentation/esp32_datasheet_en_0.pdf" H 5700 2800 50  0001 C CNN
 	1    5700 2800
@@
 F 0 "C20" H 1965 3246 50  0000 L CNN
 F 1 "C" H 1965 3155 50  0000 L CNN
-F 2 "" H 1888 3050 50  0001 C CNN
+F 2 "Capacitor_SMD:C_01005_0402Metric" H 1888 3050 50  0001 C CNN
 F 3 "~" H 1850 3200 50  0001 C CNN
 	1    1850 3200
@@
 F 0 "C22" H 2665 3246 50  0000 L CNN
 F 1 "C" H 2665 3155 50  0000 L CNN
-F 2 "" H 2588 3050 50  0001 C CNN
+F 2 "Capacitor_SMD:C_01005_0402Metric" H 2588 3050 50  0001 C CNN
 F 3 "~" H 2550 3200 50  0001 C CNN
 	1    2550 3200
@@
 F 0 "C21" V 1948 2900 50  0000 C CNN
 F 1 "5.6pF" V 2039 2900 50  0000 C CNN
-F 2 "" H 2238 2750 50  0001 C CNN
+F 2 "Capacitor_SMD:C_01005_0402Metric" H 2238 2750 50  0001 C CNN
 F 3 "~" H 2200 2900 50  0001 C CNN
 	1    2200 2900
@@
 F 0 "C26" H 5515 1296 50  0000 L CNN
 F 1 "C" H 5515 1205 50  0000 L CNN
-F 2 "" H 5438 1100 50  0001 C CNN
+F 2 "Capacitor_SMD:C_0201_0603Metric" H 5438 1100 50  0001 C CNN
 F 3 "~" H 5400 1250 50  0001 C CNN
 	1    5400 1250
@@
 F 0 "C27" H 5915 1296 50  0000 L CNN
 F 1 "C" H 5915 1205 50  0000 L CNN
-F 2 "" H 5838 1100 50  0001 C CNN
+F 2 "Capacitor_SMD:C_01005_0402Metric" H 5838 1100 50  0001 C CNN
 F 3 "~" H 5800 1250 50  0001 C CNN
 	1    5800 1250
@@
 F 0 "C23" V 3598 3200 50  0000 C CNN
 F 1 "270pF" V 3689 3200 50  0000 C CNN
-F 2 "" H 3888 3050 50  0001 C CNN
+F 2 "Capacitor_SMD:C_01005_0402Metric" H 3888 3050 50  0001 C CNN
 F 3 "~" H 3850 3200 50  0001 C CNN
 	1    3850 3200
@@
 F 0 "C24" V 4000 3500 50  0000 C CNN
 F 1 "270pF" V 4100 3500 50  0000 C CNN
-F 2 "" H 3888 3350 50  0001 C CNN
+F 2 "Capacitor_SMD:C_01005_0402Metric" H 3888 3350 50  0001 C CNN
 F 3 "~" H 3850 3500 50  0001 C CNN
 	1    3850 3500
@@
 F 0 "R36" H 10470 5296 50  0000 L CNN
 F 1 "10K" H 10470 5205 50  0000 L CNN
-F 2 "" V 10330 5250 50  0001 C CNN
+F 2 "Resistor_SMD:R_01005_0402Metric" V 10330 5250 50  0001 C CNN
 F 3 "~" H 10400 5250 50  0001 C CNN
 	1    10400 5250
@@
 F 0 "R29" V 9693 5600 50  0000 C CNN
 F 1 "0R" V 9784 5600 50  0000 C CNN
-F 2 "" V 9830 5600 50  0001 C CNN
+F 2 "Resistor_SMD:R_01005_0402Metric" V 9830 5600 50  0001 C CNN
 F 3 "~" H 9900 5600 50  0001 C CNN
 	1    9900 5600
@@
 F 0 "SW2" H 9250 6135 50  0000 C CNN
 F 1 "SW_Push" H 9250 6044 50  0000 C CNN
-F 2 "" H 9250 6050 50  0001 C CNN
+F 2 "Button_Switch_SMD:SW_Push_1P1T_NO_6x6mm_H9.5mm" H 9250 6050 50  0001 C CNN
 F 3 "~" H 9250 6050 50  0001 C CNN
 	1    9250 5850
@@
 F 0 "C28" H 10515 5996 50  0000 L CNN
 F 1 "1uF" H 10515 5905 50  0000 L CNN
-F 2 "" H 10438 5800 50  0001 C CNN
+F 2 "Capacitor_SMD:C_01005_0402Metric" H 10438 5800 50  0001 C CNN
 F 3 "~" H 10400 5950 50  0001 C CNN
 	1    10400 5950
@@
 F 0 "H1" H 8900 796 50  0000 L CNN
 F 1 "MountingHole" H 8900 705 50  0000 L CNN
-F 2 "" H 8800 750 50  0001 C CNN
+F 2 "Fiducial:Fiducial_1mm_Mask2mm" H 8800 750 50  0001 C CNN
 F 3 "~" H 8800 750 50  0001 C CNN
 	1    8800 750
@@
 F 0 "H2" H 9650 796 50  0000 L CNN
 F 1 "MountingHole" H 9650 705 50  0000 L CNN
-F 2 "" H 9550 750 50  0001 C CNN
+F 2 "Fiducial:Fiducial_1mm_Mask2mm" H 9550 750 50  0001 C CNN
 F 3 "~" H 9550 750 50  0001 C CNN
 	1    9550 750
@@
 F 0 "R23" V 1300 900 50  0000 C CNN
 F 1 "470" V 1200 900 50  0000 C CNN
-F 2 "" V 1330 900 50  0001 C CNN
+F 2 "Resistor_SMD:R_01005_0402Metric" V 1330 900 50  0001 C CNN
 F 3 "~" H 1400 900 50  0001 C CNN
 	1    1400 900
@@
 F 0 "R22" V 1600 750 50  0000 C CNN
 F 1 "470" V 1500 750 50  0000 C CNN
-F 2 "" V 1330 750 50  0001 C CNN
+F 2 "Resistor_SMD:R_01005_0402Metric" V 1330 750 50  0001 C CNN
 F 3 "~" H 1400 750 50  0001 C CNN
 	1    1400 750
@@
 F 0 "R33" V 10050 2350 50  0000 C CNN
 F 1 "22" V 9950 2350 50  0000 C CNN
-F 2 "" V 10080 2350 50  0001 C CNN
+F 2 "Resistor_SMD:R_01005_0402Metric" V 10080 2350 50  0001 C CNN
 F 3 "~" H 10150 2350 50  0001 C CNN
 	1    10150 2350
@@
 F 0 "R32" V 10350 2200 50  0000 C CNN
 F 1 "22" V 10250 2200 50  0000 C CNN
-F 2 "" V 10080 2200 50  0001 C CNN
+F 2 "Resistor_SMD:R_01005_0402Metric" V 10080 2200 50  0001 C CNN
 F 3 "~" H 10150 2200 50  0001 C CNN
 	1    10150 2200
@@
 F 0 "R31" V 10050 1650 50  0000 C CNN
 F 1 "22" V 9950 1650 50  0000 C CNN
-F 2 "" V 10080 1650 50  0001 C CNN
+F 2 "Resistor_SMD:R_01005_0402Metric" V 10080 1650 50  0001 C CNN
 F 3 "~" H 10150 1650 50  0001 C CNN
 	1    10150 1650
@@
 F 0 "R30" V 10350 1500 50  0000 C CNN
 F 1 "22" V 10250 1500 50  0000 C CNN
-F 2 "" V 10080 1500 50  0001 C CNN
+F 2 "Resistor_SMD:R_01005_0402Metric" V 10080 1500 50  0001 C CNN
 F 3 "~" H 10150 1500 50  0001 C CNN
 	1    10150 1500
@@
 F 0 "D13" H 9643 4016 50  0000 C CNN
 F 1 "LED RED" H 9643 3925 50  0000 C CNN
-F 2 "" H 9650 3800 50  0001 C CNN
+F 2 "LED_SMD:LED_0201_0603Metric" H 9650 3800 50  0001 C CNN
 F 3 "~" H 9650 3800 50  0001 C CNN
 	1    9650 3800
@@
 F 0 "R34" V 10150 3800 50  0000 C CNN
 F 1 "2K" V 10050 3800 50  0000 C CNN
-F 2 "" V 10180 3800 50  0001 C CNN
+F 2 "Resistor_SMD:R_01005_0402Metric" V 10180 3800 50  0001 C CNN
 F 3 "~" H 10250 3800 50  0001 C CNN
 	1    10250 3800
@@
 F 0 "D14" H 9643 4616 50  0000 C CNN
 F 1 "LED GREEN" H 9643 4525 50  0000 C CNN
-F 2 "" H 9650 4400 50  0001 C CNN
+F 2 "LED_SMD:LED_0201_0603Metric" H 9650 4400 50  0001 C CNN
 F 3 "~" H 9650 4400 50  0001 C CNN
 	1    9650 4400
@@
 F 0 "R35" V 10150 4400 50  0000 C CNN
 F 1 "2K" V 10050 4400 50  0000 C CNN
-F 2 "" V 10180 4400 50  0001 C CNN
+F 2 "Resistor_SMD:R_01005_0402Metric" V 10180 4400 50  0001 C CNN
 F 3 "~" H 10250 4400 50  0001 C CNN
 	1    10250 4400
@@
 F 0 "D9" H 4150 7266 50  0000 C CNN
 F 1 "ULC0511C" H 4150 7175 50  0000 C CNN
-F 2 "" H 4150 7050 50  0001 C CNN
+F 2 "Diode_SMD:D_01005_0402Metric" H 4150 7050 50  0001 C CNN
 F 3 "~" H 4150 7050 50  0001 C CNN
 	1    4150 7050
@@
 F 0 "D12" H 6300 7266 50  0000 C CNN
 F 1 "ULC0511C" H 6300 7175 50  0000 C CNN
-F 2 "" H 6300 7050 50  0001 C CNN
+F 2 "Diode_SMD:D_01005_0402Metric" H 6300 7050 50  0001 C CNN
 F 3 "~" H 6300 7050 50  0001 C CNN
 	1    6300 7050
@@
 F 0 "R26" V 4900 7050 50  0000 C CNN
 F 1 "NC" V 4800 7050 50  0000 C CNN
-F 2 "" V 4930 7050 50  0001 C CNN
+F 2 "Resistor_SMD:R_01005_0402Metric" V 4930 7050 50  0001 C CNN
 F 3 "~" H 5000 7050 50  0001 C CNN
 	1    5000 7050
@@
 F 0 "R27" V 5200 7050 50  0000 C CNN
 F 1 "NC" V 5100 7050 50  0000 C CNN
-F 2 "" V 5230 7050 50  0001 C CNN
+F 2 "Resistor_SMD:R_01005_0402Metric" V 5230 7050 50  0001 C CNN
 F 3 "~" H 5300 7050 50  0001 C CNN
 	1    5300 7050
@@
 F 0 "R28" V 5500 7050 50  0000 C CNN
 F 1 "NC" V 5400 7050 50  0000 C CNN
-F 2 "" V 5530 7050 50  0001 C CNN
+F 2 "Resistor_SMD:R_01005_0402Metric" V 5530 7050 50  0001 C CNN
 F 3 "~" H 5600 7050 50  0001 C CNN
 	1    5600 7050
@@
 F 0 "D10" H 4450 7266 50  0000 C CNN
 F 1 "ULC0511C" H 4450 7175 50  0000 C CNN
-F 2 "" H 4450 7050 50  0001 C CNN
+F 2 "Diode_SMD:D_01005_0402Metric" H 4450 7050 50  0001 C CNN
 F 3 "~" H 4450 7050 50  0001 C CNN
 	1    4450 7050
@@
 F 0 "D11" H 5950 7266 50  0000 C CNN
 F 1 "ULC0511C" H 5950 7175 50  0000 C CNN
-F 2 "" H 5950 7050 50  0001 C CNN
+F 2 "Diode_SMD:D_01005_0402Metric" H 5950 7050 50  0001 C CNN
 F 3 "~" H 5950 7050 50  0001 C CNN
 	1    5950 7050
@@
 F 0 "J4" H 1050 7750 50  0000 L CNN
 F 1 "Conn_01x13_Female" H 1000 7650 50  0000 L CNN
-F 2 "" H 1550 6900 50  0001 C CNN
+F 2 "TerminalBlock_Phoenix:TerminalBlock_Phoenix_PT-1,5-13-5.0-H_1x13_P5.00mm_Horizontal" H 1550 6900 50  0001 C CNN
 F 3 "~" H 1550 6900 50  0001 C CNN
 	1    1550 6900
@@
 F 0 "J5" H 1900 6200 50  0000 L CNN
 F 1 "Conn_01x13_Female" H 1250 6100 50  0000 L CNN
-F 2 "" H 2000 6900 50  0001 C CNN
+F 2 "TerminalBlock_Phoenix:TerminalBlock_Phoenix_PT-1,5-13-5.0-H_1x13_P5.00mm_Horizontal" H 2000 6900 50  0001 C CNN
 F 3 "~" H 2000 6900 50  0001 C CNN
 	1    2000 6900
@@
 F 0 "J3" H 1400 5767 50  0000 C CNN
 F 1 "Micro_SD_Card" H 1400 5676 50  0000 C CNN
-F 2 "" H 2600 5350 50  0001 C CNN
+F 2 "Connector_Card:microSD_HC_Hirose_DM3D-SF" H 2600 5350 50  0001 C CNN
 F 3 "http://katalog.we-online.de/em/datasheet/693072010801.pdf" H 1450 5050 50  0001 C CNN
 	1    1450 5050
@@
 F 0 "H3" H 10400 796 50  0000 L CNN
 F 1 "MountingHole" H 10400 705 50  0000 L CNN
-F 2 "" H 10300 750 50  0001 C CNN
+F 2 "Fiducial:Fiducial_1mm_Mask2mm" H 10300 750 50  0001 C CNN
 F 3 "~" H 10300 750 50  0001 C CNN
 	1    10300 750
@@
 F 0 "D8" H 3400 4466 50  0000 C CNN
 F 1 "ULC0511C" H 3400 4375 50  0000 C CNN
-F 2 "" H 3400 4250 50  0001 C CNN
+F 2 "Diode_SMD:D_01005_0402Metric" H 3400 4250 50  0001 C CNN
 F 3 "~" H 3400 4250 50  0001 C CNN
 	1    3400 4250
@@
 F 0 "R25" V 2800 4400 50  0000 C CNN
 F 1 "NC" V 2700 4400 50  0000 C CNN
-F 2 "" V 2830 4400 50  0001 C CNN
+F 2 "Resistor_SMD:R_01005_0402Metric" V 2830 4400 50  0001 C CNN
 F 3 "~" H 2900 4400 50  0001 C CNN
 	1    2900 4400
@@
 F 0 "C25" H 4115 5296 50  0000 L CNN
 F 1 "C" H 4115 5205 50  0000 L CNN
-F 2 "" H 4038 5100 50  0001 C CNN
+F 2 "Capacitor_SMD:C_01005_0402Metric" H 4038 5100 50  0001 C CNN
 F 3 "~" H 4000 5250 50  0001 C CNN
 	1    4000 5250
@@
 F 0 "D7" H 2400 5866 50  0000 C CNN
 F 1 "ULC0511C" H 2400 5775 50  0000 C CNN
-F 2 "" H 2400 5650 50  0001 C CNN
+F 2 "Diode_SMD:D_01005_0402Metric" H 2400 5650 50  0001 C CNN
 F 3 "~" H 2400 5650 50  0001 C CNN
 	1    2400 5650
@@
 F 0 "R24" V 2700 5650 50  0000 C CNN
 F 1 "NC" V 2800 5650 50  0000 C CNN
-F 2 "" V 2530 5650 50  0001 C CNN
+F 2 "Resistor_SMD:R_01005_0402Metric" V 2530 5650 50  0001 C CNN
 F 3 "~" H 2600 5650 50  0001 C CNN
 	1    2600 5650

Commit message: Comienzo PCB
Parts:
- AE3: value Antenna_Chip -> Pcb_Antenna; footprint (none) -> MyAntennas:SWRA117D
Connections:
- net +3.3VP: now also J4.11 (Pin_11); no longer J4.3 (Pin_3)
- net +5V: now also J4.13 (Pin_13); no longer J4.1 (Pin_1)
- net GND: now also J4.10 (Pin_10), J4.12 (Pin_12); no longer J4.2 (Pin_2), J4.4 (Pin_4)
- net HPDIO1: now also J4.8 (Pin_8); no longer J4.6 (Pin_6)
- net IO19: now also J4.6 (Pin_6); no longer J4.8 (Pin_8)
- net IO21: now also J4.1 (Pin_1); no longer J4.13 (Pin_13)
- net IO22: now also J4.4 (Pin_4); no longer J4.10 (Pin_10)
- net IO23: now also J4.5 (Pin_5); no longer J4.9 (Pin_9)
- net RXD: now also J4.3 (Pin_3); no longer J4.11 (Pin_11)
- net TXD: now also J4.2 (Pin_2); no longer J4.12 (Pin_12)
Changed lines of the file:
@@
 encoding utf-8
 Sheet 5 5
-Title ""
-Date ""
-Rev ""
-Comp ""
-Comment1 ""
+Title "TTGO"
+Date "2019-07-05"
+Rev "Rev 1.0"
+Comp "Ing. Hernán Dario Ferreyra- Revisor: Suarez Sebastian Alejandro"
+Comment1 "Rediseño basado en TTGO-LORA32-V2.0 (https://github.com/LilyGO/TTGO-LORA32-V2.0)"
 Comment2 ""
 Comment3 ""
@@
 P 1250 3000
 F 0 "AE3" V 1567 3081 50  0000 C CNN
-F 1 "Antenna_Chip" V 1476 3081 50  0000 C CNN
-F 2 "" H 1150 3175 50  0001 C CNN
+F 1 "Pcb_Antenna" V 1476 3081 50  0000 C CNN
+F 2 "MyAntennas:SWRA117D" H 1150 3175 50  0001 C CNN
 F 3 "~" H 1150 3175 50  0001 C CNN
 	1    1250 3000
@@
 F 3 "~" H 1550 6900 50  0001 C CNN
 	1    1550 6900
-	1    0    0    -1
-$EndComp
-$Comp
+	1    0    0    1
+$EndComp
+$Comp
