File: ReadaptTTGO/microesp32.sch (KiCad schematic (older format))
At the start: 42 parts, among them J3 Micro_SD_Card, J4 Conn_01x13_Female, J5 Conn_01x13_Female, SW2 SW_Push, U2 ESP32

Commit message: Entrega revision 1.2
Connections:
- net +3V3: now also R26.1, R27.1, R28.1; no longer R26.2, R27.2, R28.2
- net CLK-SCK-IO14: now also R27.2; no longer R27.1
- net SD0-MISO-IO2: now also R28.2; no longer R28.1
- net SD3-CS-IO13: now also R26.2; no longer R26.1
Other:
- note added: "Microcontrolador principal y Outputs."
- note added: "Pin sin especificar, ignorar error."
- moved on the sheet: C25
Changed lines of the file:
@@
 	6150 7500 6150 7450
 Connection ~ 6150 7450
-$Comp
-L Device:R R26
-U 1 1 5D328144
-P 5000 7050
-F 0 "R26" V 4900 7050 50  0000 C CNN
-F 1 "NC" V 4800 7050 50  0000 C CNN
-F 2 "Resistor_SMD:R_01005_0402Metric" V 4930 7050 50  0001 C CNN
-F 3 "~" H 5000 7050 50  0001 C CNN
-	1    5000 7050
-	1    0    0    -1
-$EndComp
 Wire Wire Line
 	3400 6150 5600 6150
 Wire Wire Line
 	3400 6250 5300 6250
-$Comp
-L Device:R R27
-U 1 1 5D342FBD
-P 5300 7050
-F 0 "R27" V 5200 7050 50  0000 C CNN
-F 1 "NC" V 5100 7050 50  0000 C CNN
-F 2 "Resistor_SMD:R_01005_0402Metric" V 5230 7050 50  0001 C CNN
-F 3 "~" H 5300 7050 50  0001 C CNN
-	1    5300 7050
-	1    0    0    -1
-$EndComp
-$Comp
-L Device:R R28
-U 1 1 5D34367A
-P 5600 7050
-F 0 "R28" V 5500 7050 50  0000 C CNN
-F 1 "NC" V 5400 7050 50  0000 C CNN
-F 2 "Resistor_SMD:R_01005_0402Metric" V 5530 7050 50  0001 C CNN
-F 3 "~" H 5600 7050 50  0001 C CNN
-	1    5600 7050
-	1    0    0    -1
-$EndComp
 Wire Wire Line
 	4450 6650 5000 6650
-Wire Wire Line
-	5000 6650 5000 6900
 Connection ~ 4450 6650
 Wire Wire Line
 	4450 6650 4450 6900
-Wire Wire Line
-	5300 6900 5300 6250
 Connection ~ 5300 6250
-Wire Wire Line
-	5600 6900 5600 6150
 Connection ~ 5600 6150
 Wire Wire Line
 	5300 6250 5950 6250
-Wire Wire Line
-	5000 7200 5000 7600
-Wire Wire Line
-	5000 7600 5300 7600
-Wire Wire Line
-	5600 7600 5600 7200
-Wire Wire Line
-	5300 7200 5300 7600
-Connection ~ 5300 7600
-Wire Wire Line
-	5300 7600 5600 7600
-$Comp
-L power:+3V3 #PWR0177
-U 1 1 5D36FAE7
-P 5750 7600
-F 0 "#PWR0177" H 5750 7450 50  0001 C CNN
-F 1 "+3V3" H 5765 7773 50  0000 C CNN
-F 2 "" H 5750 7600 50  0001 C CNN
-F 3 "" H 5750 7600 50  0001 C CNN
-	1    5750 7600
-	1    0    0    -1
-$EndComp
-Wire Wire Line
-	5750 7600 5600 7600
-Connection ~ 5600 7600
 Connection ~ 5950 6250
 $Comp
@@
 L power:GND #PWR0183
 U 1 1 5D9A23A9
-P 3400 4000
-F 0 "#PWR0183" H 3400 3750 50  0001 C CNN
-F 1 "GND" H 3405 3827 50  0000 C CNN
-F 2 "" H 3400 4000 50  0001 C CNN
-F 3 "" H 3400 4000 50  0001 C CNN
-	1    3400 4000
-	-1   0    0    1
+P 4300 4550
+F 0 "#PWR0183" H 4300 4300 50  0001 C CNN
+F 1 "GND" H 4305 4377 50  0000 C CNN
+F 2 "" H 4300 4550 50  0001 C CNN
+F 3 "" H 4300 4550 50  0001 C CNN
+	1    4300 4550
+	1    0    0    -1
 $EndComp
 Wire Wire Line
@@
 	3400 4400 3400 4650
 Wire Wire Line
-	2350 5050 4000 5050
-$Comp
-L power:+3V3 #PWR0185
-U 1 1 5DA7263A
-P 4100 4800
-F 0 "#PWR0185" H 4100 4650 50  0001 C CNN
-F 1 "+3V3" H 4115 4973 50  0000 C CNN
-F 2 "" H 4100 4800 50  0001 C CNN
-F 3 "" H 4100 4800 50  0001 C CNN
-	1    4100 4800
-	1    0    0    -1
-$EndComp
-Wire Wire Line
-	4100 4800 4100 5050
+	2350 5050 3600 5050
 $Comp
 L Device:C C25
 U 1 1 5DA7CDD1
-P 4000 5250
-F 0 "C25" H 4115 5296 50  0000 L CNN
-F 1 "C" H 4115 5205 50  0000 L CNN
-F 2 "Capacitor_SMD:C_01005_0402Metric" H 4038 5100 50  0001 C CNN
-F 3 "~" H 4000 5250 50  0001 C CNN
-	1    4000 5250
+P 3600 5250
+F 0 "C25" H 3715 5296 50  0000 L CNN
+F 1 "C" H 3715 5205 50  0000 L CNN
+F 2 "Capacitor_SMD:C_01005_0402Metric" H 3638 5100 50  0001 C CNN
+F 3 "~" H 3600 5250 50  0001 C CNN
+	1    3600 5250
 	1    0    0    -1
 $EndComp
@@
 L power:GND #PWR0186
 U 1 1 5DA88977
-P 4000 5450
-F 0 "#PWR0186" H 4000 5200 50  0001 C CNN
-F 1 "GND" H 4005 5277 50  0000 C CNN
-F 2 "" H 4000 5450 50  0001 C CNN
-F 3 "" H 4000 5450 50  0001 C CNN
-	1    4000 5450
-	1    0    0    -1
-$EndComp
-Wire Wire Line
-	4000 5450 4000 5400
-Wire Wire Line
-	4000 5100 4000 5050
-Connection ~ 4000 5050
-Wire Wire Line
-	4000 5050 4100 5050
+P 3600 5450
+F 0 "#PWR0186" H 3600 5200 50  0001 C CNN
+F 1 "GND" H 3605 5277 50  0000 C CNN
+F 2 "" H 3600 5450 50  0001 C CNN
+F 3 "" H 3600 5450 50  0001 C CNN
+	1    3600 5450
+	1    0    0    -1
+$EndComp
+Wire Wire Line
+	3600 5450 3600 5400
 $Comp
 L Device:D_TVS D?
@@
 L power:+3V3 #PWR0188
 U 1 1 5DB56193
-P 2600 5850
-F 0 "#PWR0188" H 2600 5700 50  0001 C CNN
-F 1 "+3V3" H 2615 6023 50  0000 C CNN
-F 2 "" H 2600 5850 50  0001 C CNN
-F 3 "" H 2600 5850 50  0001 C CNN
-	1    2600 5850
-	-1   0    0    1
+P 4150 5550
+F 0 "#PWR0188" H 4150 5400 50  0001 C CNN
+F 1 "+3V3" H 4165 5723 50  0000 C CNN
+F 2 "" H 4150 5550 50  0001 C CNN
+F 3 "" H 4150 5550 50  0001 C CNN
+	1    4150 5550
+	1    0    0    -1
 $EndComp
 Wire Wire Line
@@
 $EndComp
 $Comp
-L power:GND #PWR?
+L power:GND #PWR0148
 U 1 1 5D5A9AF7
 P 8800 4000
-F 0 "#PWR?" H 8800 3750 50  0001 C CNN
+F 0 "#PWR0148" H 8800 3750 50  0001 C CNN
 F 1 "GND" H 8805 3827 50  0000 C CNN
 F 2 "" H 8800 4000 50  0001 C CNN
@@
 Wire Wire Line
 	8800 3900 8800 4000
+Text Notes 4000 2750 0    50   ~ 0
+Pin sin especificar, ignorar error.
+Wire Wire Line
+	3600 5100 3600 5050
+Connection ~ 3600 5050
+Wire Wire Line
+	3600 5050 3700 5050
+$Comp
+L power:+3V3 #PWR0185
+U 1 1 5DA7263A
+P 3700 4800
+F 0 "#PWR0185" H 3700 4650 50  0001 C CNN
+F 1 "+3V3" H 3715 4973 50  0000 C CNN
+F 2 "" H 3700 4800 50  0001 C CNN
+F 3 "" H 3700 4800 50  0001 C CNN
+	1    3700 4800
+	1    0    0    -1
+$EndComp
+Wire Wire Line
+	3700 5050 3700 4800
+Wire Wire Line
+	4300 4550 4300 4000
+Wire Wire Line
+	4300 4000 3400 4000
+Wire Wire Line
+	4150 5550 4150 5850
+Wire Wire Line
+	4150 5850 2600 5850
+$Comp
+L Device:R R26
+U 1 1 5D3B7A65
+P 5000 5800
+F 0 "R26" V 4900 5800 50  0000 C CNN
+F 1 "NC" V 4800 5800 50  0000 C CNN
+F 2 "Resistor_SMD:R_01005_0402Metric" V 4930 5800 50  0001 C CNN
+F 3 "~" H 5000 5800 50  0001 C CNN
+	1    5000 5800
+	1    0    0    -1
+$EndComp
+$Comp
+L Device:R R27
+U 1 1 5D3B7A6D
+P 5300 5800
+F 0 "R27" V 5200 5800 50  0000 C CNN
+F 1 "NC" V 5100 5800 50  0000 C CNN
+F 2 "Resistor_SMD:R_01005_0402Metric" V 5230 5800 50  0001 C CNN
+F 3 "~" H 5300 5800 50  0001 C CNN
+	1    5300 5800
+	1    0    0    -1
+$EndComp
+$Comp
+L Device:R R28
+U 1 1 5D3B7A73
+P 5600 5800
+F 0 "R28" V 5500 5800 50  0000 C CNN
+F 1 "NC" V 5400 5800 50  0000 C CNN
+F 2 "Resistor_SMD:R_01005_0402Metric" V 5530 5800 50  0001 C CNN
+F 3 "~" H 5600 5800 50  0001 C CNN
+	1    5600 5800
+	1    0    0    -1
+$EndComp
+$Comp
+L power:+3V3 #PWR?
+U 1 1 5D3B7A88
+P 5300 5500
+F 0 "#PWR?" H 5300 5350 50  0001 C CNN
+F 1 "+3V3" H 5315 5673 50  0000 C CNN
+F 2 "" H 5300 5500 50  0001 C CNN
+F 3 "" H 5300 5500 50  0001 C CNN
+	1    5300 5500
+	1    0    0    -1
+$EndComp
+Wire Wire Line
+	5600 6150 5600 5950
+Wire Wire Line
+	5300 6250 5300 5950
+Wire Wire Line
+	5000 6650 5000 5950
+Wire Wire Line
+	5300 5500 5300 5550
+Wire Wire Line
+	5300 5550 5000 5550
+Wire Wire Line
+	5000 5550 5000 5650
+Wire Wire Line
+	5300 5550 5300 5650
+Connection ~ 5300 5550
+Wire Wire Line
+	5300 5550 5600 5550
+Wire Wire Line
+	5600 5550 5600 5650
+Text Notes 2800 750  0    157  ~ 0
+Microcontrolador principal y Outputs.
 $EndSCHEMATC
