File: ReadaptTTGO/Alimentacionsch.sch (KiCad schematic (older format))
At the start: 12 parts

Commit message: Primer aproximacion.
Parts:
- added C? (x5): 100nF, symbol Device:C
- added C? (x3): 10uF, symbol Device:C
- added D?: LED, symbol Device:LED
- added D?: 2A FUSE, symbol Device:D
- added D?: BS5819, symbol Device:D
- added J?: USB_B_Micro, symbol Connector:USB_B_Micro
- added R? (x6): 100K, symbol Device:R
- added R? (x2): 2K, symbol Device:R
- D? (x2): value D_TVS -> ULC0511C
- FL?: value EMI_Filter_LL_1423 -> EMI_Filter_ACM2012
Connections:
- net at U?.1 (STAT): now also D?.1 (K)
- net GND: now reaches U?.2 (VSS)
- net GND: now also D?.1 (A1), D?.2 (A2), J?.1 (Pin_1), J?.SH (Shield), U?.2 (GND), U?.2 (GND), U?.2 (GND), U?.25 (GND), C?.2, C?.2, C?.2, C?.2, C?.2, C?.2, C?.2, C?.2, J?.5 (GND), J?.6 (Shield), R?.2, R?.2, R?.2
- net +BATT: now reaches U?.3 (VBAT)
- net +BATT: now also J?.2 (Pin_2), C?.1, D?.2 (A), R?.1, R?.1
- net VBUS: now reaches U?.4 (VDD)
- net VBUS: now also C?.1, D?.2 (A), J?.1 (VBUS), R?.1
- net at U?.5 (PROG): now also R?.1
- net RTS: now reaches U?.19 (RTS)
- net RTS: now also U?.1 (DTr1_Emitter), U?.5 (DTr2_Base)
- net U0TXD: now reaches U?.20 (RXD)
- net U0RXD: now reaches U?.21 (TXD)
- net DTR: now reaches U?.23 (DTR)
- net DTR: now also U?.2 (DTr1_Base), U?.4 (DTr2_Emitter)
- net DP: now reaches U?.3 (D+)
- net DP: now also FL?.3, R?.2
- net DM: now reaches U?.4 (D-)
- net DM: now also FL?.4, R?.2
- net +3.3VP: now reaches U?.5 (VIO)
- net +3.3VP: now also U?.5 (VOUT), U?.6 (VDD), U?.7 (REGIN), C?.1, C?.1, C?.1
- net +5V: now reaches U?.8 (VBUS)
- net +5V: now also SW?.1 (A), U?.1 (VIN), U?.1 (VIN), C?.1, C?.1, R?.1, R?.1
- net IO0: now reaches U?.3 (DTr2_Collector)
- net RST_EN: now reaches U?.6 (DTr1_Collector)
- net at U?.3 (ON/~OFF~): now also R?.2 (x2)
- net +3V3: now reaches U?.5 (VOUT)
- net +3V3: now also C?.1
- net D-: now reaches FL?.1
- net D-: now also D?.1 (A1), R?.1, J?.2 (D-)
- net D+: now reaches FL?.2
- net D+: now also D?.2 (A2), R?.1, J?.3 (D+)
- net +5VD: now reaches SW?.2 (B)
- net +5VD: now also D?.1 (K), D?.1 (K)
- new net: D?.2 (A), R?.2
- new net IO35: R?.1, R?.1, R?.2, R?.2
Other:
- moved on the sheet: D?, FL?, J?, R?, SW?, U?

Commit message: Anotacciones
Parts:
- gave numbers to parts that had none: 32
Connections:
- no-connect marks 0 -> 2

Commit message: ERC completo
Connections:
- no-connect marks 2 -> 15
Other:
- moved on the sheet: D3, D4, SW1
Changed lines of the file:
@@
-$EndComp
-$Comp
-L Regulator_Linear:LP2985-5.0 U6
-U 1 1 5D0BD25C
-P 9850 2350
-F 0 "U6" H 9850 2692 50  0000 C CNN
-F 1 "ME6211" H 9850 2601 50  0000 C CNN
-F 2 "Package_TO_SOT_SMD:SOT-23-5" H 9850 2675 50  0001 C CNN
-F 3 "http://www.ti.com/lit/ds/symlink/lp2985.pdf" H 9850 2350 50  0001 C CNN
-	1    9850 2350
-	1    0    0    -1
 $EndComp
 $Comp
@@
 L power:+5V #PWR0112
 U 1 1 5D2CDE73
-P 8250 1050
-F 0 "#PWR0112" H 8250 900 50  0001 C CNN
-F 1 "+5V" H 8265 1223 50  0000 C CNN
-F 2 "" H 8250 1050 50  0001 C CNN
-F 3 "" H 8250 1050 50  0001 C CNN
-	1    8250 1050
+P 8200 1050
+F 0 "#PWR0112" H 8200 900 50  0001 C CNN
+F 1 "+5V" H 8215 1223 50  0000 C CNN
+F 2 "" H 8200 1050 50  0001 C CNN
+F 3 "" H 8200 1050 50  0001 C CNN
+	1    8200 1050
 	1    0    0    -1
 $EndComp
@@
 	8350 1150 8350 1050
 Wire Wire Line
-	8250 1050 8350 1050
-Connection ~ 8350 1050
-Wire Wire Line
-	8350 1050 8600 1050
-Wire Wire Line
 	8600 1150 8600 1050
-Connection ~ 8600 1050
 $Comp
 L power:+3.3VP #PWR0114
@@
 	8600 2350 8600 2250
 Connection ~ 8600 2250
-Wire Wire Line
-	8600 2250 9400 2250
 $Comp
 L Device:C C8
@@
 L power:+5VD #PWR0121
 U 1 1 5D34BFFF
-P 4200 1200
-F 0 "#PWR0121" H 4200 1050 50  0001 C CNN
-F 1 "+5VD" H 4215 1373 50  0000 C CNN
-F 2 "" H 4200 1200 50  0001 C CNN
-F 3 "" H 4200 1200 50  0001 C CNN
-	1    4200 1200
+P 5100 1100
+F 0 "#PWR0121" H 5100 950 50  0001 C CNN
+F 1 "+5VD" H 5115 1273 50  0000 C CNN
+F 2 "" H 5100 1100 50  0001 C CNN
+F 3 "" H 5100 1100 50  0001 C CNN
+	1    5100 1100
 	1    0    0    -1
 $EndComp
@@
 L Device:D D3
 U 1 1 5D35DA3E
-P 3050 1000
-F 0 "D3" H 3200 950 50  0000 C CNN
-F 1 "2A FUSE" H 2950 1100 50  0000 C CNN
-F 2 "" H 3050 1000 50  0001 C CNN
-F 3 "~" H 3050 1000 50  0001 C CNN
-	1    3050 1000
+P 2950 1000
+F 0 "D3" H 3100 950 50  0000 C CNN
+F 1 "2A FUSE" H 3000 1100 50  0000 C CNN
+F 2 "" H 2950 1000 50  0001 C CNN
+F 3 "~" H 2950 1000 50  0001 C CNN
+	1    2950 1000
 	-1   0    0    1
 $EndComp
@@
 L Device:D D4
 U 1 1 5D35E64A
-P 3050 1350
-F 0 "D4" H 3200 1300 50  0000 C CNN
-F 1 "BS5819" H 2950 1450 50  0000 C CNN
-F 2 "" H 3050 1350 50  0001 C CNN
-F 3 "~" H 3050 1350 50  0001 C CNN
-	1    3050 1350
+P 2950 1350
+F 0 "D4" H 3100 1300 50  0000 C CNN
+F 1 "BS5819" H 3000 1450 50  0000 C CNN
+F 2 "" H 2950 1350 50  0001 C CNN
+F 3 "~" H 2950 1350 50  0001 C CNN
+	1    2950 1350
 	-1   0    0    1
 $EndComp
 Wire Wire Line
-	4750 1300 4850 1300
-Wire Wire Line
-	4350 1200 4200 1200
-Wire Wire Line
-	4850 1100 4750 1100
+	5650 1200 5750 1200
+Wire Wire Line
+	5250 1100 5100 1100
+Wire Wire Line
+	5750 1000 5650 1000
 $Comp
 L power:+5V #PWR0122
 U 1 1 5D3429C9
-P 4850 1100
-F 0 "#PWR0122" H 4850 950 50  0001 C CNN
-F 1 "+5V" H 4865 1273 50  0000 C CNN
-F 2 "" H 4850 1100 50  0001 C CNN
-F 3 "" H 4850 1100 50  0001 C CNN
-	1    4850 1100
+P 5750 1000
+F 0 "#PWR0122" H 5750 850 50  0001 C CNN
+F 1 "+5V" H 5765 1173 50  0000 C CNN
+F 2 "" H 5750 1000 50  0001 C CNN
+F 3 "" H 5750 1000 50  0001 C CNN
+	1    5750 1000
 	1    0    0    -1
 $EndComp
@@
 L Switch:SW_SPDT SW1
 U 1 1 5D0C8BD6
-P 4550 1200
-F 0 "SW1" H 4550 1485 50  0000 C CNN
-F 1 "SW_SPDT" H 4550 1394 50  0000 C CNN
-F 2 "" H 4550 1200 50  0001 C CNN
-F 3 "~" H 4550 1200 50  0001 C CNN
-	1    4550 1200
-	1    0    0    -1
-$EndComp
-Wire Wire Line
-	2900 1350 2650 1350
-Wire Wire Line
-	2900 1000 2650 1000
-Wire Wire Line
-	3200 1000 3450 1000
-Wire Wire Line
-	3200 1350 3450 1350
+P 5450 1100
+F 0 "SW1" H 5450 1385 50  0000 C CNN
+F 1 "SW_SPDT" H 5450 1294 50  0000 C CNN
+F 2 "" H 5450 1100 50  0001 C CNN
+F 3 "~" H 5450 1100 50  0001 C CNN
+	1    5450 1100
+	1    0    0    -1
+$EndComp
+Wire Wire Line
+	2800 1350 2550 1350
+Wire Wire Line
+	2800 1000 2550 1000
+Wire Wire Line
+	3100 1000 3200 1000
 $Comp
 L power:+5VD #PWR0123
 U 1 1 5D380740
-P 3450 1000
-F 0 "#PWR0123" H 3450 850 50  0001 C CNN
-F 1 "+5VD" H 3465 1173 50  0000 C CNN
-F 2 "" H 3450 1000 50  0001 C CNN
-F 3 "" H 3450 1000 50  0001 C CNN
-	1    3450 1000
+P 3600 1000
+F 0 "#PWR0123" H 3600 850 50  0001 C CNN
+F 1 "+5VD" H 3615 1173 50  0000 C CNN
+F 2 "" H 3600 1000 50  0001 C CNN
+F 3 "" H 3600 1000 50  0001 C CNN
+	1    3600 1000
 	1    0    0    -1
 $EndComp
@@
 L power:+5VD #PWR0124
 U 1 1 5D383C1F
-P 3450 1350
-F 0 "#PWR0124" H 3450 1200 50  0001 C CNN
-F 1 "+5VD" H 3465 1523 50  0000 C CNN
-F 2 "" H 3450 1350 50  0001 C CNN
-F 3 "" H 3450 1350 50  0001 C CNN
-	1    3450 1350
+P 3600 1350
+F 0 "#PWR0124" H 3600 1200 50  0001 C CNN
+F 1 "+5VD" H 3615 1523 50  0000 C CNN
+F 2 "" H 3600 1350 50  0001 C CNN
+F 3 "" H 3600 1350 50  0001 C CNN
+	1    3600 1350
 	1    0    0    -1
 $EndComp
@@
 L power:VBUS #PWR0125
 U 1 1 5D38EF45
-P 2650 1000
-F 0 "#PWR0125" H 2650 850 50  0001 C CNN
-F 1 "VBUS" H 2665 1173 50  0000 C CNN
-F 2 "" H 2650 1000 50  0001 C CNN
-F 3 "" H 2650 1000 50  0001 C CNN
-	1    2650 1000
+P 2550 1000
+F 0 "#PWR0125" H 2550 850 50  0001 C CNN
+F 1 "VBUS" H 2565 1173 50  0000 C CNN
+F 2 "" H 2550 1000 50  0001 C CNN
+F 3 "" H 2550 1000 50  0001 C CNN
+	1    2550 1000
 	1    0    0    -1
 $EndComp
@@
 L power:+BATT #PWR0126
 U 1 1 5D399996
-P 2650 1350
-F 0 "#PWR0126" H 2650 1200 50  0001 C CNN
-F 1 "+BATT" H 2665 1523 50  0000 C CNN
-F 2 "" H 2650 1350 50  0001 C CNN
-F 3 "" H 2650 1350 50  0001 C CNN
-	1    2650 1350
+P 2550 1350
+F 0 "#PWR0126" H 2550 1200 50  0001 C CNN
+F 1 "+BATT" H 2565 1523 50  0000 C CNN
+F 2 "" H 2550 1350 50  0001 C CNN
+F 3 "" H 2550 1350 50  0001 C CNN
+	1    2550 1350
 	1    0    0    -1
 $EndComp
@@
 IO35
 $Comp
-L power:PWR_FLAG #FLG?
-U 1 1 5DD0EBB0
-P 9400 2250
-F 0 "#FLG?" H 9400 2325 50  0001 C CNN
-F 1 "PWR_FLAG" H 9400 2423 50  0000 C CNN
-F 2 "" H 9400 2250 50  0001 C CNN
-F 3 "~" H 9400 2250 50  0001 C CNN
-	1    9400 2250
-	1    0    0    -1
-$EndComp
-Connection ~ 9400 2250
-Wire Wire Line
-	9400 2250 9450 2250
-Wire Wire Line
-	8600 1050 9250 1050
-$Comp
-L power:PWR_FLAG #FLG?
+L power:PWR_FLAG #FLG0102
 U 1 1 5DD0F952
-P 9250 1050
-F 0 "#FLG?" H 9250 1125 50  0001 C CNN
-F 1 "PWR_FLAG" H 9250 1223 50  0000 C CNN
-F 2 "" H 9250 1050 50  0001 C CNN
-F 3 "~" H 9250 1050 50  0001 C CNN
-	1    9250 1050
-	1    0    0    -1
-$EndComp
-Connection ~ 9250 1050
-Wire Wire Line
-	9250 1050 9450 1050
+P 3200 1000
+F 0 "#FLG0102" H 3200 1075 50  0001 C CNN
+F 1 "PWR_FLAG" H 3200 1173 50  0000 C CNN
+F 2 "" H 3200 1000 50  0001 C CNN
+F 3 "~" H 3200 1000 50  0001 C CNN
+	1    3200 1000
+	1    0    0    -1
+$EndComp
 NoConn ~ 10250 1150
 NoConn ~ 10250 2350
+NoConn ~ 3100 4250
+NoConn ~ 3100 4150
+NoConn ~ 3100 4050
+NoConn ~ 3100 3950
+NoConn ~ 3100 3750
+NoConn ~ 3100 3550
+NoConn ~ 3100 3050
+NoConn ~ 3100 3150
+NoConn ~ 1900 3450
+NoConn ~ 1900 3350
+NoConn ~ 1900 3050
+$Comp
+L Regulator_Linear:LP2985-5.0 U6
+U 1 1 5D0BD25C
+P 9850 2350
+F 0 "U6" H 9850 2692 50  0000 C CNN
+F 1 "ME6211" H 9850 2601 50  0000 C CNN
+F 2 "Package_TO_SOT_SMD:SOT-23-5" H 9850 2675 50  0001 C CNN
+F 3 "http://www.ti.com/lit/ds/symlink/lp2985.pdf" H 9850 2350 50  0001 C CNN
+	1    9850 2350
+	1    0    0    -1
+$EndComp
+Wire Wire Line
+	8600 2250 9450 2250
+NoConn ~ 1150 1300
+NoConn ~ 5750 1200
+Connection ~ 3200 1000
+$Comp
+L power:PWR_FLAG #FLG0101
+U 1 1 5DE495DA
+P 8600 1050
+F 0 "#FLG0101" H 8600 1125 50  0001 C CNN
+F 1 "PWR_FLAG" H 8600 1223 50  0000 C CNN
+F 2 "" H 8600 1050 50  0001 C CNN
+F 3 "~" H 8600 1050 50  0001 C CNN
+	1    8600 1050
+	1    0    0    -1
+$EndComp
+Wire Wire Line
+	3200 1000 3600 1000
+Wire Wire Line
+	8200 1050 8350 1050
+Wire Wire Line
+	8600 1050 9450 1050
+Wire Wire Line
+	3100 1350 3600 1350
+Wire Wire Line
+	8350 1050 8600 1050
+Connection ~ 8350 1050
+Connection ~ 8600 1050
 $EndSCHEMATC

Commit message: Añadidos Footprints
Parts:
- C1, C3, C6: footprint (none) -> Capacitor_SMD:C_0201_0603Metric
- C2, C4, C5, C7, C8: footprint (none) -> Capacitor_SMD:C_01005_0402Metric
- D1, D2: footprint (none) -> Diode_SMD:D_01005_0402Metric
- D3, D4: footprint (none) -> Diode_SMD:D_SOD-123
- D5: footprint (none) -> LED_SMD:LED_0201_0603Metric
- FL1: footprint (none) -> Filter:Filter_Bourns_SRF0905_6.0x9.2mm
- J1: footprint (none) -> Connector_USB:USB_Micro-B_Amphenol_10103594-0001LF_Horizontal
- J2: footprint (none) -> Connector_BarrelJack:BarrelJack_Wuerth_6941xx301002
- R1, R10, R2, R3, R4, R5, R6, R7, R8, R9: footprint (none) -> Resistor_SMD:R_01005_0402Metric
- SW1: footprint (none) -> Button_Switch_THT:SW_CuK_OS102011MA1QN1_SPDT_Angled
Changed lines of the file:
@@
 F 0 "FL1" H 2000 6431 50  0000 C CNN
 F 1 "EMI_Filter_ACM2012" H 2000 6340 50  0000 C CNN
-F 2 "" H 2000 5900 50  0001 C CNN
+F 2 "Filter:Filter_Bourns_SRF0905_6.0x9.2mm" H 2000 5900 50  0001 C CNN
 F 3 "~" V 2000 6190 50  0001 C CNN
 	1    2000 6150
@@
 F 0 "J2" H 10800 4700 50  0000 L CNN
 F 1 "Conn_01x02_Shielded" H 10350 4850 50  0000 L CNN
-F 2 "" H 10650 4700 50  0001 C CNN
+F 2 "Connector_BarrelJack:BarrelJack_Wuerth_6941xx301002" H 10650 4700 50  0001 C CNN
 F 3 "~" H 10650 4700 50  0001 C CNN
 	1    10650 4700
@@
 F 0 "D1" H 1300 7016 50  0000 C CNN
 F 1 "ULC0511C" H 1300 6925 50  0000 C CNN
-F 2 "" H 1300 6800 50  0001 C CNN
+F 2 "Diode_SMD:D_01005_0402Metric" H 1300 6800 50  0001 C CNN
 F 3 "~" H 1300 6800 50  0001 C CNN
 	1    1300 6800
@@
 F 0 "D2" H 1700 7016 50  0000 C CNN
 F 1 "ULC0511C" H 1700 6925 50  0000 C CNN
-F 2 "" H 1700 6800 50  0001 C CNN
+F 2 "Diode_SMD:D_01005_0402Metric" H 1700 6800 50  0001 C CNN
 F 3 "~" H 1700 6800 50  0001 C CNN
 	1    1700 6800
@@
 F 0 "R2" H 2070 6496 50  0000 L CNN
 F 1 "R" H 2070 6405 50  0000 L CNN
-F 2 "" V 1930 6450 50  0001 C CNN
+F 2 "Resistor_SMD:R_01005_0402Metric" V 1930 6450 50  0001 C CNN
 F 3 "~" H 2000 6450 50  0001 C CNN
 	1    2000 6450
@@
 F 0 "R1" H 2070 5796 50  0000 L CNN
 F 1 "R" H 2070 5705 50  0000 L CNN
-F 2 "" V 1930 5750 50  0001 C CNN
+F 2 "Resistor_SMD:R_01005_0402Metric" V 1930 5750 50  0001 C CNN
 F 3 "~" H 2000 5750 50  0001 C CNN
 	1    2000 5750
@@
 F 0 "R5" H 7270 5296 50  0000 L CNN
 F 1 "2K" H 7270 5205 50  0000 L CNN
-F 2 "" V 7130 5250 50  0001 C CNN
+F 2 "Resistor_SMD:R_01005_0402Metric" V 7130 5250 50  0001 C CNN
 F 3 "~" H 7200 5250 50  0001 C CNN
 	1    7200 5250
@@
 F 0 "C6" H 9065 5346 50  0000 L CNN
 F 1 "10uF" H 9065 5255 50  0000 L CNN
-F 2 "" H 8988 5150 50  0001 C CNN
+F 2 "Capacitor_SMD:C_0201_0603Metric" H 8988 5150 50  0001 C CNN
 F 3 "~" H 8950 5300 50  0001 C CNN
 	1    8950 5300
@@
 F 0 "R10" H 9820 5496 50  0000 L CNN
 F 1 "100K" H 9820 5405 50  0000 L CNN
-F 2 "" V 9680 5450 50  0001 C CNN
+F 2 "Resistor_SMD:R_01005_0402Metric" V 9680 5450 50  0001 C CNN
 F 3 "~" H 9750 5450 50  0001 C CNN
 	1    9750 5450
@@
 F 0 "R9" H 9820 5096 50  0000 L CNN
 F 1 "100K" H 9820 5005 50  0000 L CNN
-F 2 "" V 9680 5050 50  0001 C CNN
+F 2 "Resistor_SMD:R_01005_0402Metric" V 9680 5050 50  0001 C CNN
 F 3 "~" H 9750 5050 50  0001 C CNN
 	1    9750 5050
@@
 F 0 "C3" V 7348 4300 50  0000 C CNN
 F 1 "10uF" V 7439 4300 50  0000 C CNN
-F 2 "" H 7638 4150 50  0001 C CNN
+F 2 "Capacitor_SMD:C_0201_0603Metric" H 7638 4150 50  0001 C CNN
 F 3 "~" H 7600 4300 50  0001 C CNN
 	1    7600 4300
@@
 F 0 "R6" H 8320 4346 50  0000 L CNN
 F 1 "2K" H 8320 4255 50  0000 L CNN
-F 2 "" V 8180 4300 50  0001 C CNN
+F 2 "Resistor_SMD:R_01005_0402Metric" V 8180 4300 50  0001 C CNN
 F 3 "~" H 8250 4300 50  0001 C CNN
 	1    8250 4300
@@
 F 0 "D5" V 8489 4433 50  0000 R CNN
 F 1 "LED" V 8398 4433 50  0000 R CNN
-F 2 "" H 8450 4550 50  0001 C CNN
+F 2 "LED_SMD:LED_0201_0603Metric" H 8450 4550 50  0001 C CNN
 F 3 "~" H 8450 4550 50  0001 C CNN
 	1    8450 4550
@@
 F 0 "R7" V 8900 1100 50  0000 L CNN
 F 1 "100K" V 8800 1050 50  0000 L CNN
-F 2 "" V 8930 1150 50  0001 C CNN
+F 2 "Resistor_SMD:R_01005_0402Metric" V 8930 1150 50  0001 C CNN
 F 3 "~" H 9000 1150 50  0001 C CNN
 	1    9000 1150
@@
 F 0 "C4" H 8465 1346 50  0000 L CNN
 F 1 "100nF" H 8465 1255 50  0000 L CNN
-F 2 "" H 8388 1150 50  0001 C CNN
+F 2 "Capacitor_SMD:C_01005_0402Metric" H 8388 1150 50  0001 C CNN
 F 3 "~" H 8350 1300 50  0001 C CNN
 	1    8350 1300
@@
 F 0 "C7" H 10915 1246 50  0000 L CNN
 F 1 "100nF" H 10915 1155 50  0000 L CNN
-F 2 "" H 10838 1050 50  0001 C CNN
+F 2 "Capacitor_SMD:C_01005_0402Metric" H 10838 1050 50  0001 C CNN
 F 3 "~" H 10800 1200 50  0001 C CNN
 	1    10800 1200
@@
 F 0 "R8" V 8900 2300 50  0000 L CNN
 F 1 "100K" V 8800 2250 50  0000 L CNN
-F 2 "" V 8930 2350 50  0001 C CNN
+F 2 "Resistor_SMD:R_01005_0402Metric" V 8930 2350 50  0001 C CNN
 F 3 "~" H 9000 2350 50  0001 C CNN
 	1    9000 2350
@@
 F 0 "C5" H 8465 2546 50  0000 L CNN
 F 1 "100nF" H 8465 2455 50  0000 L CNN
-F 2 "" H 8388 2350 50  0001 C CNN
+F 2 "Capacitor_SMD:C_01005_0402Metric" H 8388 2350 50  0001 C CNN
 F 3 "~" H 8350 2500 50  0001 C CNN
 	1    8350 2500
@@
 F 0 "C8" H 10915 2446 50  0000 L CNN
 F 1 "100nF" H 10915 2355 50  0000 L CNN
-F 2 "" H 10838 2250 50  0001 C CNN
+F 2 "Capacitor_SMD:C_01005_0402Metric" H 10838 2250 50  0001 C CNN
 F 3 "~" H 10800 2400 50  0001 C CNN
 	1    10800 2400
@@
 F 0 "D3" H 3100 950 50  0000 C CNN
 F 1 "2A FUSE" H 3000 1100 50  0000 C CNN
-F 2 "" H 2950 1000 50  0001 C CNN
+F 2 "Diode_SMD:D_SOD-123" H 2950 1000 50  0001 C CNN
 F 3 "~" H 2950 1000 50  0001 C CNN
 	1    2950 1000
@@
 F 0 "D4" H 3100 1300 50  0000 C CNN
 F 1 "BS5819" H 3000 1450 50  0000 C CNN
-F 2 "" H 2950 1350 50  0001 C CNN
+F 2 "Diode_SMD:D_SOD-123" H 2950 1350 50  0001 C CNN
 F 3 "~" H 2950 1350 50  0001 C CNN
 	1    2950 1350
@@
 F 0 "SW1" H 5450 1385 50  0000 C CNN
 F 1 "SW_SPDT" H 5450 1294 50  0000 C CNN
-F 2 "" H 5450 1100 50  0001 C CNN
+F 2 "Button_Switch_THT:SW_CuK_OS102011MA1QN1_SPDT_Angled" H 5450 1100 50  0001 C CNN
 F 3 "~" H 5450 1100 50  0001 C CNN
 	1    5450 1100
@@
 F 0 "C2" H 4015 2796 50  0000 L CNN
 F 1 "10uF" H 4015 2705 50  0000 L CNN
-F 2 "" H 3938 2600 50  0001 C CNN
+F 2 "Capacitor_SMD:C_01005_0402Metric" H 3938 2600 50  0001 C CNN
 F 3 "~" H 3900 2750 50  0001 C CNN
 	1    3900 2750
@@
 F 0 "C1" H 3565 2796 50  0000 L CNN
 F 1 "100nF" H 3565 2705 50  0000 L CNN
-F 2 "" H 3488 2600 50  0001 C CNN
+F 2 "Capacitor_SMD:C_0201_0603Metric" H 3488 2600 50  0001 C CNN
 F 3 "~" H 3450 2750 50  0001 C CNN
 	1    3450 2750
@@
 F 0 "J1" H 907 1567 50  0000 C CNN
 F 1 "USB_B_Micro" H 907 1476 50  0000 C CNN
-F 2 "" H 1000 1050 50  0001 C CNN
+F 2 "Connector_USB:USB_Micro-B_Amphenol_10103594-0001LF_Horizontal" H 1000 1050 50  0001 C CNN
 F 3 "~" H 1000 1050 50  0001 C CNN
 	1    850  1100
@@
 F 0 "R3" H 4570 5946 50  0000 L CNN
 F 1 "100K" H 4570 5855 50  0000 L CNN
-F 2 "" V 4430 5900 50  0001 C CNN
+F 2 "Resistor_SMD:R_01005_0402Metric" V 4430 5900 50  0001 C CNN
 F 3 "~" H 4500 5900 50  0001 C CNN
 	1    4500 5900
@@
 F 0 "R4" H 4570 6596 50  0000 L CNN
 F 1 "100K" H 4570 6505 50  0000 L CNN
-F 2 "" V 4430 6550 50  0001 C CNN
+F 2 "Resistor_SMD:R_01005_0402Metric" V 4430 6550 50  0001 C CNN
 F 3 "~" H 4500 6550 50  0001 C CNN
 	1    4500 6550

Commit message: Comienzo PCB
Parts:
- U3: footprint (none) -> Package_TO_SOT_SMD:SOT-563
Other:
- moved on the sheet: C1
Changed lines of the file:
@@
 encoding utf-8
 Sheet 2 5
-Title ""
-Date ""
-Rev ""
-Comp ""
-Comment1 ""
+Title "TTGO"
+Date "2019-07-05"
+Rev "Rev 1.0"
+Comp "Ing. Hernán Dario Ferreyra- Revisor: Suarez Sebastian Alejandro"
+Comment1 "Rediseño basado en TTGO-LORA32-V2.0 (https://github.com/LilyGO/TTGO-LORA32-V2.0)"
 Comment2 ""
 Comment3 ""
@@
 F 0 "U3" H 6550 2315 50  0000 C CNN
 F 1 "EMH3" H 6550 2224 50  0000 C CNN
-F 2 "" H 6000 2200 50  0001 C CNN
+F 2 "Package_TO_SOT_SMD:SOT-563" H 6000 2200 50  0001 C CNN
 F 3 "" H 6000 2200 50  0001 C CNN
 	1    6000 2050
@@
 	1    0    0    -1
 $EndComp
-Wire Wire Line
-	3450 2900 3900 2900
-Connection ~ 3450 2600
-Wire Wire Line
-	3450 2600 3900 2600
 $Comp
 L power:+3.3VP #PWR0127
@@
 Wire Wire Line
 	2400 2750 2400 2400
-Wire Wire Line
-	2500 2400 2500 2500
 $Comp
 L power:+3.3VP #PWR0128
 U 1 1 5D294858
-P 2450 2400
-F 0 "#PWR0128" H 2600 2350 50  0001 C CNN
-F 1 "+3.3VP" H 2470 2543 50  0000 C CNN
-F 2 "" H 2450 2400 50  0001 C CNN
-F 3 "" H 2450 2400 50  0001 C CNN
-	1    2450 2400
-	1    0    0    -1
-$EndComp
-Wire Wire Line
-	2400 2400 2450 2400
-Connection ~ 2450 2400
-Wire Wire Line
-	2450 2400 2500 2400
-Connection ~ 2500 2500
+P 2400 2400
+F 0 "#PWR0128" H 2550 2350 50  0001 C CNN
+F 1 "+3.3VP" H 2420 2543 50  0000 C CNN
+F 2 "" H 2400 2400 50  0001 C CNN
+F 3 "" H 2400 2400 50  0001 C CNN
+	1    2400 2400
+	1    0    0    -1
+$EndComp
 Wire Wire Line
 	3100 3250 3450 3250
@@
 Wire Wire Line
 	3100 3650 3450 3650
-Connection ~ 3900 2900
-Wire Wire Line
-	3900 2950 3900 2900
-Wire Wire Line
-	3450 2500 3450 2600
-Wire Wire Line
-	2500 2500 3450 2500
-Wire Wire Line
-	2500 2500 2500 2750
+Wire Wire Line
+	3600 2400 3600 2500
 Wire Wire Line
 	1550 3500 1550 3650
@@
 $EndComp
 $Comp
-L Device:C C2
-U 1 1 5D1CAA22
-P 3900 2750
-F 0 "C2" H 4015 2796 50  0000 L CNN
-F 1 "10uF" H 4015 2705 50  0000 L CNN
-F 2 "Capacitor_SMD:C_01005_0402Metric" H 3938 2600 50  0001 C CNN
-F 3 "~" H 3900 2750 50  0001 C CNN
-	1    3900 2750
-	1    0    0    -1
-$EndComp
-$Comp
-L power:GND #PWR0129
-U 1 1 5D1C9C40
-P 3900 2950
-F 0 "#PWR0129" H 3900 2700 50  0001 C CNN
-F 1 "GND" H 3905 2777 50  0000 C CNN
-F 2 "" H 3900 2950 50  0001 C CNN
-F 3 "" H 3900 2950 50  0001 C CNN
-	1    3900 2950
-	1    0    0    -1
-$EndComp
-$Comp
 L Device:C C1
 U 1 1 5D1C5E8C
-P 3450 2750
-F 0 "C1" H 3565 2796 50  0000 L CNN
-F 1 "100nF" H 3565 2705 50  0000 L CNN
-F 2 "Capacitor_SMD:C_0201_0603Metric" H 3488 2600 50  0001 C CNN
-F 3 "~" H 3450 2750 50  0001 C CNN
-	1    3450 2750
+P 3250 2700
+F 0 "C1" H 3365 2746 50  0000 L CNN
+F 1 "100nF" H 3365 2655 50  0000 L CNN
+F 2 "Capacitor_SMD:C_0201_0603Metric" H 3288 2550 50  0001 C CNN
+F 3 "~" H 3250 2700 50  0001 C CNN
+	1    3250 2700
 	1    0    0    -1
 $EndComp
@@
 Connection ~ 8350 1050
 Connection ~ 8600 1050
+Connection ~ 2500 2400
+Wire Wire Line
+	2500 2400 2500 2750
+$Comp
+L power:GND #PWR0129
+U 1 1 5D1C9C40
+P 3900 3050
+F 0 "#PWR0129" H 3900 2800 50  0001 C CNN
+F 1 "GND" H 3905 2877 50  0000 C CNN
+F 2 "" H 3900 3050 50  0001 C CNN
+F 3 "" H 3900 3050 50  0001 C CNN
+	1    3900 3050
+	1    0    0    -1
+$EndComp
+Wire Wire Line
+	3900 2950 3900 2900
+$Comp
+L Device:C C2
+U 1 1 5D1CAA22
+P 3900 2750
+F 0 "C2" H 4000 2850 50  0000 L CNN
+F 1 "10uF" H 4000 2750 50  0000 L CNN
+F 2 "Capacitor_SMD:C_01005_0402Metric" H 3938 2600 50  0001 C CNN
+F 3 "~" H 3900 2750 50  0001 C CNN
+	1    3900 2750
+	1    0    0    -1
+$EndComp
+Wire Wire Line
+	3900 3050 3900 2950
+Connection ~ 3900 2950
+Wire Wire Line
+	3250 2950 3250 2850
+Wire Wire Line
+	3250 2950 3900 2950
+Wire Wire Line
+	3250 2550 3250 2500
+Wire Wire Line
+	3900 2500 3900 2600
+Connection ~ 3600 2500
+Wire Wire Line
+	3600 2500 3900 2500
+Wire Wire Line
+	3250 2500 3600 2500
+Wire Wire Line
+	2500 2400 3600 2400
+Connection ~ 2400 2400
+Wire Wire Line
+	2400 2400 2500 2400
 $EndSCHEMATC

Commit message: Entrega revision 1.2
Other:
- note added: "Circuitos de bateria y alimentacion electrica."
- moved on the sheet: D3, D4, J1, SW1, U3
