File: ReadaptTTGO/moduloRF.sch (KiCad schematic (older format))
At the start: 1 part

Commit message: Primer aproximacion.
Parts:
- added AE?: Antenna Jack, symbol Device:Antenna_Shield
- added AE?: WIFI ANT, symbol Device:Antenna_Chip
- added C?: 220pF, symbol Device:C
- added C? (x2): C, symbol Device:C
- added R?: R, symbol Device:R
- added R?: 0R, symbol Device:R
Connections:
- net GND: now reaches U?.1 (GND)
- net GND: now also U?.10 (GND), U?.8 (GND), AE?.1 (A), AE?.2 (PCB_Trace), C?.2, C?.2
- net +3.3VP: now reaches U?.13 (3.3V)
- net IO26: now reaches U?.14 (DIO0)
- net HPDIO1: now reaches U?.15 (DIO1)
- net HPDIO2: now reaches U?.16 (DIO2)
- net IO19: now reaches U?.2 (MISO)
- net IO27: now reaches U?.3 (MOSI)
- net IO5: now reaches U?.4 (SCK)
- net IO18: now reaches U?.5 (NSS)
- net IO23: now reaches U?.6 (RESET)
- net ANT: now reaches U?.9 (ANT)
- net ANT: now also C?.1, C?.2
- new net: AE?.2 (Shield), R?.2
- new net: AE?.1 (FEED), R?.2
- new net: C?.1, C?.1, R?.1, R?.1
Other:
- note added: "IO23=RESET\nIO18=NSS/SEL\nIO5=SCK\nIO27=MOSI/SDI\nIO19=MISO/SDO\nIO26=DI0/IO0"
- moved on the sheet: U?

Commit message: Anotacciones
Parts:
- gave numbers to parts that had none: 8
Changed lines of the file:
@@
 $EndDescr
 $Comp
-L RF_Module:RFM69HCW U?
+L RF_Module:RFM69HCW U9
 U 1 1 5D0A7BFB
 P 2150 2650
-F 0 "U?" H 1750 3350 50  0000 C CNN
+F 0 "U9" H 1750 3350 50  0000 C CNN
 F 1 "RFM69HCW" H 1900 3250 50  0000 C CNN
 F 2 "" H -1150 4300 50  0001 C CNN
@@
 $EndComp
 $Comp
-L power:GND #PWR?
+L power:GND #PWR0154
 U 1 1 5D5049C8
 P 2150 3400
-F 0 "#PWR?" H 2150 3150 50  0001 C CNN
+F 0 "#PWR0154" H 2150 3150 50  0001 C CNN
 F 1 "GND" H 2155 3227 50  0000 C CNN
 F 2 "" H 2150 3400 50  0001 C CNN
@@
 P 2150 2000
 AR Path="/5D087535/5D50AD9D" Ref="#PWR?"  Part="1"
-AR Path="/5D086661/5D50AD9D" Ref="#PWR?"  Part="1"
-F 0 "#PWR?" H 2300 1950 50  0001 C CNN
+AR Path="/5D086661/5D50AD9D" Ref="#PWR0155"  Part="1"
+F 0 "#PWR0155" H 2300 1950 50  0001 C CNN
 F 1 "+3.3VP" H 2170 2143 50  0000 C CNN
 F 2 "" H 2150 2000 50  0001 C CNN
@@
 IO19
 $Comp
-L Device:Antenna_Shield AE?
+L Device:Antenna_Shield AE1
 U 1 1 5D51F020
 P 3900 5850
-F 0 "AE?" V 3978 6080 50  0000 L CNN
+F 0 "AE1" V 3978 6080 50  0000 L CNN
 F 1 "Antenna Jack" V 3887 6080 50  0000 L CNN
 F 2 "" H 3900 5950 50  0001 C CNN
@@
 $EndComp
 $Comp
-L Device:Antenna_Chip AE?
+L Device:Antenna_Chip AE2
 U 1 1 5D51FFE1
 P 4400 5300
-F 0 "AE?" V 4372 5605 50  0000 L CNN
+F 0 "AE2" V 4372 5605 50  0000 L CNN
 F 1 "WIFI ANT" V 4463 5605 50  0000 L CNN
 F 2 "" H 4300 5475 50  0001 C CNN
@@
 $EndComp
 $Comp
-L Device:C C?
+L Device:C C18
 U 1 1 5D5238B0
 P 2550 5200
-F 0 "C?" V 2298 5200 50  0000 C CNN
+F 0 "C18" V 2298 5200 50  0000 C CNN
 F 1 "220pF" V 2389 5200 50  0000 C CNN
 F 2 "" H 2588 5050 50  0001 C CNN
@@
 $EndComp
 $Comp
-L Device:C C?
+L Device:C C19
 U 1 1 5D524DEE
 P 2900 5500
-F 0 "C?" H 3015 5546 50  0000 L CNN
+F 0 "C19" H 3015 5546 50  0000 L CNN
 F 1 "C" H 3015 5455 50  0000 L CNN
 F 2 "" H 2938 5350 50  0001 C CNN
@@
 $EndComp
 $Comp
-L Device:C C?
+L Device:C C17
 U 1 1 5D5279A1
 P 2250 5500
-F 0 "C?" H 2365 5546 50  0000 L CNN
+F 0 "C17" H 2365 5546 50  0000 L CNN
 F 1 "C" H 2365 5455 50  0000 L CNN
 F 2 "" H 2288 5350 50  0001 C CNN
@@
 $EndComp
 $Comp
-L Device:R R?
+L Device:R R20
 U 1 1 5D528D84
 P 3700 5550
-F 0 "R?" H 3770 5596 50  0000 L CNN
+F 0 "R20" H 3770 5596 50  0000 L CNN
 F 1 "R" H 3770 5505 50  0000 L CNN
 F 2 "" V 3630 5550 50  0001 C CNN
@@
 	2900 5900 2250 5900
 $Comp
-L power:GND #PWR?
+L power:GND #PWR0156
 U 1 1 5D52C9D5
 P 2900 5950
-F 0 "#PWR?" H 2900 5700 50  0001 C CNN
+F 0 "#PWR0156" H 2900 5700 50  0001 C CNN
 F 1 "GND" H 2905 5777 50  0000 C CNN
 F 2 "" H 2900 5950 50  0001 C CNN
@@
 ANT
 $Comp
-L Device:R R?
+L Device:R R21
 U 1 1 5D531E22
 P 3900 5200
-F 0 "R?" V 4107 5200 50  0000 C CNN
+F 0 "R21" V 4107 5200 50  0000 C CNN
 F 1 "0R" V 4016 5200 50  0000 C CNN
 F 2 "" V 3830 5200 50  0001 C CNN
@@
 	4050 5200 4300 5200
 $Comp
-L power:GND #PWR?
+L power:GND #PWR0157
 U 1 1 5D538F07
 P 4300 5550
-F 0 "#PWR?" H 4300 5300 50  0001 C CNN
+F 0 "#PWR0157" H 4300 5300 50  0001 C CNN
 F 1 "GND" H 4305 5377 50  0000 C CNN
 F 2 "" H 4300 5550 50  0001 C CNN
@@
 	4300 5400 4300 5550
 $Comp
-L power:GND #PWR?
+L power:GND #PWR0158
 U 1 1 5D53D17D
 P 3700 5950
-F 0 "#PWR?" H 3700 5700 50  0001 C CNN
+F 0 "#PWR0158" H 3700 5700 50  0001 C CNN
 F 1 "GND" H 3705 5777 50  0000 C CNN
 F 2 "" H 3700 5950 50  0001 C CNN

Commit message: ERC completo
Connections:
- no-connect marks 0 -> 3
Changed lines of the file:
@@
 Text Notes 5800 2850 0    50   ~ 0
 IO23=RESET\nIO18=NSS/SEL\nIO5=SCK\nIO27=MOSI/SDI\nIO19=MISO/SDO\nIO26=DI0/IO0
+NoConn ~ 2650 2550
+NoConn ~ 2650 2650
+NoConn ~ 2650 2750
 $EndSCHEMATC

Commit message: Añadidos Footprints
Parts:
- C17, C18, C19: footprint (none) -> Capacitor_SMD:C_01005_0402Metric
- R20, R21: footprint (none) -> Resistor_SMD:R_01005_0402Metric
Changed lines of the file:
@@
 F 0 "C18" V 2298 5200 50  0000 C CNN
 F 1 "220pF" V 2389 5200 50  0000 C CNN
-F 2 "" H 2588 5050 50  0001 C CNN
+F 2 "Capacitor_SMD:C_01005_0402Metric" H 2588 5050 50  0001 C CNN
 F 3 "~" H 2550 5200 50  0001 C CNN
 	1    2550 5200
@@
 F 0 "C19" H 3015 5546 50  0000 L CNN
 F 1 "C" H 3015 5455 50  0000 L CNN
-F 2 "" H 2938 5350 50  0001 C CNN
+F 2 "Capacitor_SMD:C_01005_0402Metric" H 2938 5350 50  0001 C CNN
 F 3 "~" H 2900 5500 50  0001 C CNN
 	1    2900 5500
@@
 F 0 "C17" H 2365 5546 50  0000 L CNN
 F 1 "C" H 2365 5455 50  0000 L CNN
-F 2 "" H 2288 5350 50  0001 C CNN
+F 2 "Capacitor_SMD:C_01005_0402Metric" H 2288 5350 50  0001 C CNN
 F 3 "~" H 2250 5500 50  0001 C CNN
 	1    2250 5500
@@
 F 0 "R20" H 3770 5596 50  0000 L CNN
 F 1 "R" H 3770 5505 50  0000 L CNN
-F 2 "" V 3630 5550 50  0001 C CNN
+F 2 "Resistor_SMD:R_01005_0402Metric" V 3630 5550 50  0001 C CNN
 F 3 "~" H 3700 5550 50  0001 C CNN
 	1    3700 5550
@@
 F 0 "R21" V 4107 5200 50  0000 C CNN
 F 1 "0R" V 4016 5200 50  0000 C CNN
-F 2 "" V 3830 5200 50  0001 C CNN
+F 2 "Resistor_SMD:R_01005_0402Metric" V 3830 5200 50  0001 C CNN
 F 3 "~" H 3900 5200 50  0001 C CNN
 	1    3900 5200

Commit message: Comienzo PCB
Parts:
- AE1: footprint (none) -> Connector_Coaxial:SMA_Amphenol_132134_Vertical
- AE2: footprint (none) -> Connector_Coaxial:SMA_Amphenol_132134-11_Vertical
- U9: footprint (none) -> RF_Module:HOPERF_RFM69HW
Connections:
- net GND: now also AE1.2 (Shield); no longer AE1.1 (A)
- net at R20.2: now also AE1.1 (A); no longer AE1.2 (Shield)
Other:
- moved on the sheet: AE1
Changed lines of the file:
@@
 encoding utf-8
 Sheet 4 5
-Title ""
-Date ""
-Rev ""
-Comp ""
-Comment1 ""
+Title "TTGO"
+Date "2019-07-05"
+Rev "Rev 1.0"
+Comp "Ing. Hernán Dario Ferreyra- Revisor: Suarez Sebastian Alejandro"
+Comment1 "Rediseño basado en TTGO-LORA32-V2.0 (https://github.com/LilyGO/TTGO-LORA32-V2.0)"
 Comment2 ""
 Comment3 ""
@@
 F 0 "U9" H 1750 3350 50  0000 C CNN
 F 1 "RFM69HCW" H 1900 3250 50  0000 C CNN
-F 2 "" H -1150 4300 50  0001 C CNN
+F 2 "RF_Module:HOPERF_RFM69HW" H -1150 4300 50  0001 C CNN
 F 3 "https://www.hoperf.com/data/upload/portal/20181127/5bfcb8284d838.pdf" H -1150 4300 50  0001 C CNN
 	1    2150 2650
@@
 L Device:Antenna_Shield AE1
 U 1 1 5D51F020
-P 3900 5850
-F 0 "AE1" V 3978 6080 50  0000 L CNN
-F 1 "Antenna Jack" V 3887 6080 50  0000 L CNN
-F 2 "" H 3900 5950 50  0001 C CNN
-F 3 "~" H 3900 5950 50  0001 C CNN
-	1    3900 5850
-	0    1    -1   0
+P 3900 5750
+F 0 "AE1" V 4150 5800 50  0000 L CNN
+F 1 "Antenna Jack" V 4050 5800 50  0000 L CNN
+F 2 "Connector_Coaxial:SMA_Amphenol_132134_Vertical" H 3900 5850 50  0001 C CNN
+F 3 "~" H 3900 5850 50  0001 C CNN
+	1    3900 5750
+	0    1    1    0
 $EndComp
 $Comp
@@
 F 0 "AE2" V 4372 5605 50  0000 L CNN
 F 1 "WIFI ANT" V 4463 5605 50  0000 L CNN
-F 2 "" H 4300 5475 50  0001 C CNN
+F 2 "Connector_Coaxial:SMA_Amphenol_132134-11_Vertical" H 4300 5475 50  0001 C CNN
 F 3 "~" H 4300 5475 50  0001 C CNN
 	1    4400 5300

Commit message: PCB sin traces
Parts:
- AE2: footprint Connector_Coaxial:SMA_Amphenol_132134-11_Vertical -> Connector_Coaxial:SMA_Amphenol_132134_Vertical
Changed lines of the file:
@@
 F 0 "AE2" V 4372 5605 50  0000 L CNN
 F 1 "WIFI ANT" V 4463 5605 50  0000 L CNN
-F 2 "Connector_Coaxial:SMA_Amphenol_132134-11_Vertical" H 4300 5475 50  0001 C CNN
+F 2 "Connector_Coaxial:SMA_Amphenol_132134_Vertical" H 4300 5475 50  0001 C CNN
 F 3 "~" H 4300 5475 50  0001 C CNN
 	1    4400 5300

Commit message: Entrega revision 1.2
Other:
- note added: "Integrado de comunicacion por radiofrecuencia."
Changed lines of the file:
@@
 NoConn ~ 2650 2650
 NoConn ~ 2650 2750
+Text Notes 1350 1300 0    197  ~ 0
+Integrado de comunicacion por radiofrecuencia.
 $EndSCHEMATC
